Commit message: description   : convert meshes to .dae

File: robots/polar_arm.xacro (robot description, xacro)
@@ -15,5 +15,5 @@
         <origin rpy="0 0 0" xyz="0 0 0"/>
         <geometry>
-          <mesh filename="package://${description_pkg}/meshes/link0.stl"/>
+          <mesh filename="package://${description_pkg}/meshes/link0.dae"/>
         </geometry>
       </visual>
@@ -21,5 +21,5 @@
         <origin rpy="0 0 0" xyz="0 0 0"/>
         <geometry>
-          <mesh filename="package://${description_pkg}/meshes/link0.stl"/>
+          <mesh filename="package://${description_pkg}/meshes/link0.dae"/>
         </geometry>
       </collision>
@@ -29,5 +29,5 @@
         <origin rpy="0 0 0" xyz="-0.0 -0.0 -0.074"/>
         <geometry>
-          <mesh filename="package://${description_pkg}/meshes/link1.stl"/>
+          <mesh filename="package://${description_pkg}/meshes/link1.dae"/>
         </geometry>
       </visual>
@@ -35,5 +35,5 @@
         <origin rpy="0 0 0" xyz="-0.0 -0.0 -0.074"/>
         <geometry>
-          <mesh filename="package://${description_pkg}/meshes/link1.stl"/>
+          <mesh filename="package://${description_pkg}/meshes/link1.dae"/>
         </geometry>
       </collision>
@@ -50,5 +50,5 @@
         <origin rpy="0 0 0" xyz="0.0 -0.0445 -0.199"/>
         <geometry>
-          <mesh filename="package://${description_pkg}/meshes/link2.stl"/>
+          <mesh filename="package://${description_pkg}/meshes/link2.dae"/>
         </geometry>
       </visual>
@@ -56,5 +56,5 @@
         <origin rpy="0 0 0" xyz="0.0 -0.0445 -0.199"/>
         <geometry>
-          <mesh filename="package://${description_pkg}/meshes/link2.stl"/>
+          <mesh filename="package://${description_pkg}/meshes/link2.dae"/>
         </geometry>
       </collision>
@@ -71,5 +71,5 @@
         <origin rpy="0 0 0" xyz="0.475211 -0.0445 -0.199"/>
         <geometry>
-          <mesh filename="package://${description_pkg}/meshes/link3.stl"/>
+          <mesh filename="package://${description_pkg}/meshes/link3.dae"/>
         </geometry>
       </visual>
@@ -77,5 +77,5 @@
         <origin rpy="0 0 0" xyz="0.475211 -0.0445 -0.199"/>
         <geometry>
-          <mesh filename="package://${description_pkg}/meshes/link3.stl"/>
+          <mesh filename="package://${description_pkg}/meshes/link3.dae"/>
         </geometry>
       </collision>
@@ -92,5 +92,5 @@
         <origin rpy="0 0 0" xyz="0.017457 -0.0 -0.300319"/>
         <geometry>
-          <mesh filename="package://${description_pkg}/meshes/link4.stl"/>
+          <mesh filename="package://${description_pkg}/meshes/link4.dae"/>
         </geometry>
       </visual>
@@ -98,5 +98,5 @@
         <origin rpy="0 0 0" xyz="0.017457 -0.0 -0.300319"/>
         <geometry>
-          <mesh filename="package://${description_pkg}/meshes/link4.stl"/>
+          <mesh filename="package://${description_pkg}/meshes/link4.dae"/>
         </geometry>
       </collision>
@@ -113,5 +113,5 @@
         <origin rpy="0 0 0" xyz="-0.110443 -0.085 -0.300319"/>
         <geometry>
-          <mesh filename="package://${description_pkg}/meshes/link5.stl"/>
+          <mesh filename="package://${description_pkg}/meshes/link5.dae"/>
         </geometry>
       </visual>
@@ -119,5 +119,5 @@
         <origin rpy="0 0 0" xyz="-0.110443 -0.085 -0.300319"/>
         <geometry>
-          <mesh filename="package://${description_pkg}/meshes/link5.stl"/>
+          <mesh filename="package://${description_pkg}/meshes/link5.dae"/>
         </geometry>
       </collision>
@@ -134,5 +134,5 @@
         <origin rpy="0 0 0" xyz="-0.155443 -0.0 -0.300319"/>
         <geometry>
-          <mesh filename="package://${description_pkg}/meshes/link6.stl"/>
+          <mesh filename="package://${description_pkg}/meshes/link6.dae"/>
         </geometry>
       </visual>
@@ -140,5 +140,5 @@
         <origin rpy="0 0 0" xyz="-0.155443 -0.0 -0.300319"/>
         <geometry>
-          <mesh filename="package://${description_pkg}/meshes/link6.stl"/>
+          <mesh filename="package://${description_pkg}/meshes/link6.dae"/>
         </geometry>
       </collision>

Commit message: description   : add joint, safety limits

File: robots/polar_arm.xacro (robot description, xacro)
@@ -11,4 +11,6 @@
       </joint>
     </xacro:unless>
+    <xacro:property name="safety_k_position" value="100.0"/>
+    <xacro:property name="safety_k_velocity" value="40.0"/>
     <link name="${arm_id}_link0">
       <visual>
@@ -40,9 +42,10 @@
     </link>
     <joint name="${arm_id}_joint1" type="revolute">
+      <safety_controller k_position="${safety_k_position}" k_velocity="${safety_k_velocity}" soft_lower_limit="${-pi}" soft_upper_limit="${pi}"/>
       <origin rpy="0 0 0" xyz="0.0 0.0 0.074"/>
       <parent link="${arm_id}_link0"/>
       <child link="${arm_id}_link1"/>
       <axis xyz="0.0 0.0 1.0"/>
-      <limit effort="87" lower="${-pi}" upper="${pi}" velocity="2.1750"/>
+      <limit effort="100" lower="${-pi}" upper="${pi}" velocity="0.1745"/> <!-- 10deg/s -->
     </joint>
     <link name="${arm_id}_link2">
@@ -61,9 +64,10 @@
     </link>
     <joint name="${arm_id}_joint2" type="revolute">
+      <safety_controller k_position="${safety_k_position}" k_velocity="${safety_k_velocity}" soft_lower_limit="${-pi}" soft_upper_limit="${pi}"/>
       <origin rpy="0 0 0" xyz="-0.0 0.0445 0.125"/>
       <parent link="${arm_id}_link1"/>
       <child link="${arm_id}_link2"/>
       <axis xyz="-0.0 1.0 -0.0"/>
-      <limit effort="87" lower="${-pi}" upper="${pi}" velocity="2.1750"/>
+      <limit effort="100" lower="${-pi}" upper="${pi}" velocity="0.1745"/> <!-- 10deg/s -->
     </joint>
     <link name="${arm_id}_link3">
@@ -82,9 +86,10 @@
     </link>
     <joint name="${arm_id}_joint3" type="revolute">
+      <safety_controller k_position="${safety_k_position}" k_velocity="${safety_k_velocity}" soft_lower_limit="${-pi}" soft_upper_limit="${pi}"/>
       <origin rpy="0 0 0" xyz="-0.475211 0.0 0.0"/>
       <parent link="${arm_id}_link2"/>
       <child link="${arm_id}_link3"/>
       <axis xyz="-0.0 -1.0 0.0"/>
-      <limit effort="87" lower="${-pi}" upper="${pi}" velocity="2.1750"/>
+      <limit effort="100" lower="${-pi}" upper="${pi}" velocity="0.1745"/> <!-- 10deg/s -->
     </joint>
     <link name="${arm_id}_link4">
@@ -103,9 +108,10 @@
     </link>
     <joint name="${arm_id}_joint4" type="revolute">
+      <safety_controller k_position="${safety_k_position}" k_velocity="${safety_k_velocity}" soft_lower_limit="${-pi}" soft_upper_limit="${pi}"/>
       <origin rpy="0 0 0" xyz="0.457754 -0.0445 0.101319"/>
       <parent link="${arm_id}_link3"/>
       <child link="${arm_id}_link4"/>
       <axis xyz="1.0 -0.0 -0.0"/>
-      <limit effort="87" lower="${-pi}" upper="${pi}" velocity="2.1750"/>
+      <limit effort="100" lower="${-pi}" upper="${pi}" velocity="0.3491"/> <!-- 20deg/s -->
     </joint>
     <link name="${arm_id}_link5">
@@ -124,9 +130,10 @@
     </link>
     <joint name="${arm_id}_joint5" type="revolute">
+      <safety_controller k_position="${safety_k_position}" k_velocity="${safety_k_velocity}" soft_lower_limit="${-pi}" soft_upper_limit="${pi}"/>
       <origin rpy="0 0 0" xyz="0.1279 0.085 0.0"/>
       <parent link="${arm_id}_link4"/>
       <child link="${arm_id}_link5"/>
       <axis xyz="0.0 -1.0 -0.0"/>
-      <limit effort="12" lower="${-pi}" upper="${pi}" velocity="2.6100"/>
+      <limit effort="100" lower="${-pi}" upper="${pi}" velocity="0.1745"/> <!-- 10deg/s -->
     </joint>
     <link name="${arm_id}_link6">
@@ -145,9 +152,10 @@
     </link>
     <joint name="${arm_id}_joint6" type="revolute">
+      <safety_controller k_position="${safety_k_position}" k_velocity="${safety_k_velocity}" soft_lower_limit="${-pi}" soft_upper_limit="${pi}"/>
       <origin rpy="0 0 0" xyz="0.045 -0.085 0.0"/>
       <parent link="${arm_id}_link5"/>
       <child link="${arm_id}_link6"/>
       <axis xyz="1.0 0.0 -0.0"/>
-      <limit effort="12" lower="${-pi}" upper="${pi}" velocity="2.6100"/>
+      <limit effort="100" lower="${-pi}" upper="${pi}" velocity="0.1745"/> <!-- 10deg/s -->
     </joint>
   </xacro:macro>

Commit message: description   : add damping, friction and safety_pos_margin

File: robots/polar_arm.xacro (robot description, xacro)
@@ -11,6 +11,9 @@
       </joint>
     </xacro:unless>
+    <xacro:property name="joint_damping" value="0.0"/>
+    <xacro:property name="joint_friction" value="0.0"/>
     <xacro:property name="safety_k_position" value="100.0"/>
     <xacro:property name="safety_k_velocity" value="40.0"/>
+    <xacro:property name="safety_pos_margin" value="0.0"/>
     <link name="${arm_id}_link0">
       <visual>
@@ -42,5 +45,5 @@
     </link>
     <joint name="${arm_id}_joint1" type="revolute">
-      <safety_controller k_position="${safety_k_position}" k_velocity="${safety_k_velocity}" soft_lower_limit="${-pi}" soft_upper_limit="${pi}"/>
+      <safety_controller k_position="${safety_k_position}" k_velocity="${safety_k_velocity}" soft_lower_limit="${-pi + safety_pos_margin}" soft_upper_limit="${pi - safety_pos_margin}"/>
       <origin rpy="0 0 0" xyz="0.0 0.0 0.074"/>
       <parent link="${arm_id}_link0"/>
@@ -48,4 +51,5 @@
       <axis xyz="0.0 0.0 1.0"/>
       <limit effort="100" lower="${-pi}" upper="${pi}" velocity="0.1745"/> <!-- 10deg/s -->
+      <dynamics damping="${joint_damping}" friction="${joint_friction}"/>
     </joint>
     <link name="${arm_id}_link2">
@@ -64,5 +68,5 @@
     </link>
     <joint name="${arm_id}_joint2" type="revolute">
-      <safety_controller k_position="${safety_k_position}" k_velocity="${safety_k_velocity}" soft_lower_limit="${-pi}" soft_upper_limit="${pi}"/>
+      <safety_controller k_position="${safety_k_position}" k_velocity="${safety_k_velocity}" soft_lower_limit="${-pi + safety_pos_margin}" soft_upper_limit="${pi - safety_pos_margin}"/>
       <origin rpy="0 0 0" xyz="-0.0 0.0445 0.125"/>
       <parent link="${arm_id}_link1"/>
@@ -70,4 +74,5 @@
       <axis xyz="-0.0 1.0 -0.0"/>
       <limit effort="100" lower="${-pi}" upper="${pi}" velocity="0.1745"/> <!-- 10deg/s -->
+      <dynamics damping="${joint_damping}" friction="${joint_friction}"/>
     </joint>
     <link name="${arm_id}_link3">
@@ -86,5 +91,5 @@
     </link>
     <joint name="${arm_id}_joint3" type="revolute">
-      <safety_controller k_position="${safety_k_position}" k_velocity="${safety_k_velocity}" soft_lower_limit="${-pi}" soft_upper_limit="${pi}"/>
+      <safety_controller k_position="${safety_k_position}" k_velocity="${safety_k_velocity}" soft_lower_limit="${-pi + safety_pos_margin}" soft_upper_limit="${pi - safety_pos_margin}"/>
       <origin rpy="0 0 0" xyz="-0.475211 0.0 0.0"/>
       <parent link="${arm_id}_link2"/>
@@ -92,4 +97,5 @@
       <axis xyz="-0.0 -1.0 0.0"/>
       <limit effort="100" lower="${-pi}" upper="${pi}" velocity="0.1745"/> <!-- 10deg/s -->
+      <dynamics damping="${joint_damping}" friction="${joint_friction}"/>
     </joint>
     <link name="${arm_id}_link4">
@@ -108,5 +114,5 @@
     </link>
     <joint name="${arm_id}_joint4" type="revolute">
-      <safety_controller k_position="${safety_k_position}" k_velocity="${safety_k_velocity}" soft_lower_limit="${-pi}" soft_upper_limit="${pi}"/>
+      <safety_controller k_position="${safety_k_position}" k_velocity="${safety_k_velocity}" soft_lower_limit="${-pi + safety_pos_margin}" soft_upper_limit="${pi - safety_pos_margin}"/>
       <origin rpy="0 0 0" xyz="0.457754 -0.0445 0.101319"/>
       <parent link="${arm_id}_link3"/>
@@ -114,4 +120,5 @@
       <axis xyz="1.0 -0.0 -0.0"/>
       <limit effort="100" lower="${-pi}" upper="${pi}" velocity="0.3491"/> <!-- 20deg/s -->
+      <dynamics damping="${joint_damping}" friction="${joint_friction}"/>
     </joint>
     <link name="${arm_id}_link5">
@@ -130,5 +137,5 @@
     </link>
     <joint name="${arm_id}_joint5" type="revolute">
-      <safety_controller k_position="${safety_k_position}" k_velocity="${safety_k_velocity}" soft_lower_limit="${-pi}" soft_upper_limit="${pi}"/>
+      <safety_controller k_position="${safety_k_position}" k_velocity="${safety_k_velocity}" soft_lower_limit="${-pi + safety_pos_margin}" soft_upper_limit="${pi - safety_pos_margin}"/>
       <origin rpy="0 0 0" xyz="0.1279 0.085 0.0"/>
       <parent link="${arm_id}_link4"/>
@@ -136,4 +143,5 @@
       <axis xyz="0.0 -1.0 -0.0"/>
       <limit effort="100" lower="${-pi}" upper="${pi}" velocity="0.1745"/> <!-- 10deg/s -->
+      <dynamics damping="${joint_damping}" friction="${joint_friction}"/>
     </joint>
     <link name="${arm_id}_link6">
@@ -152,5 +160,5 @@
     </link>
     <joint name="${arm_id}_joint6" type="revolute">
-      <safety_controller k_position="${safety_k_position}" k_velocity="${safety_k_velocity}" soft_lower_limit="${-pi}" soft_upper_limit="${pi}"/>
+      <safety_controller k_position="${safety_k_position}" k_velocity="${safety_k_velocity}" soft_lower_limit="${-pi + safety_pos_margin}" soft_upper_limit="${pi - safety_pos_margin}"/>
       <origin rpy="0 0 0" xyz="0.045 -0.085 0.0"/>
       <parent link="${arm_id}_link5"/>
@@ -158,4 +166,5 @@
       <axis xyz="1.0 0.0 -0.0"/>
       <limit effort="100" lower="${-pi}" upper="${pi}" velocity="0.1745"/> <!-- 10deg/s -->
+      <dynamics damping="${joint_damping}" friction="${joint_friction}"/>
     </joint>
   </xacro:macro>

Commit message: description   : add world joint

File: robots/polar_arm.xacro (robot description, xacro)
@@ -16,4 +16,10 @@
     <xacro:property name="safety_k_velocity" value="40.0"/>
     <xacro:property name="safety_pos_margin" value="0.0"/>
+    <link name="world" />
+    <joint name="robot_to_world" type="fixed">
+      <parent link="world" />
+      <child link="${arm_id}_link0" />
+      <origin xyz="0.0 0.0 0.0" rpy="0.0 0.0 0.0" />
+    </joint>
     <link name="${arm_id}_link0">
       <visual>

Commit message: description   : - add inertia values
Calculated in Fusion360 based on bodies.

File: robots/polar_arm.xacro (robot description, xacro)
@@ -35,4 +35,9 @@
         </geometry>
       </collision>
+      <inertial>
+        <origin rpy="0 0 0" xyz="-0.02 -0.013 0.035"/>
+        <mass value="1.0"/>
+        <inertia ixx="0.032" ixy="-0.003" ixz="0.0" iyy="0.029" iyz="0.001" izz="0.05"/>
+      </inertial>
     </link>
     <link name="${arm_id}_link1">
@@ -49,4 +54,9 @@
         </geometry>
       </collision>
+      <inertial>
+        <origin rpy="0 0 0" xyz="0.0 0.0 0.129"/>
+        <mass value="1.0"/>
+        <inertia ixx="0.006" ixy="0.0" ixz="0.0" iyy="0.005" iyz="0.0" izz="0.003"/>
+      </inertial>
     </link>
     <joint name="${arm_id}_joint1" type="revolute">
@@ -72,4 +82,9 @@
         </geometry>
       </collision>
+      <inertial>
+        <origin rpy="0 0 0" xyz="-0.238 0.0 0.19"/>
+        <mass value="1.0"/>
+        <inertia ixx="0.082" ixy="0.0" ixz="0.0" iyy="1.288" iyz="0.0" izz="1.249"/>
+      </inertial>
     </link>
     <joint name="${arm_id}_joint2" type="revolute">
@@ -95,4 +110,9 @@
         </geometry>
       </collision>
+      <inertial>
+        <origin rpy="0 0 0" xyz="0.232 0.0 0.304"/>
+        <mass value="1.0"/>
+        <inertia ixx="0.011" ixy="0.0" ixz="-0.02" iyy="0.154" iyz="0.0" izz="0.149"/>
+      </inertial>
     </link>
     <joint name="${arm_id}_joint3" type="revolute">
@@ -118,4 +138,9 @@
         </geometry>
       </collision>
+      <inertial>
+        <origin rpy="0 0 0" xyz="0.025 0.0 0.30"/>
+        <mass value="1.0"/>
+        <inertia ixx="0.019" ixy="0.0" ixz="0.0" iyy="0.008" iyz="0.0" izz="0.024"/>
+      </inertial>
     </link>
     <joint name="${arm_id}_joint4" type="revolute">
@@ -141,4 +166,9 @@
         </geometry>
       </collision>
+      <inertial>
+        <origin rpy="0 0 0" xyz="0.108 0.0 0.30"/>
+        <mass value="1.0"/>
+        <inertia ixx="0.006" ixy="0.0" ixz="0.0" iyy="0.005" iyz="0.0" izz="0.007"/>
+      </inertial>
     </link>
     <joint name="${arm_id}_joint5" type="revolute">
@@ -164,4 +194,9 @@
         </geometry>
       </collision>
+      <inertial>
+        <origin rpy="0 0 0" xyz="0.161 0.0 0.30"/>
+        <mass value="1.0"/>
+        <inertia ixx="0.0" ixy="0.0" ixz="0.0" iyy="0.0" iyz="0.0" izz="0.0"/>
+      </inertial>
     </link>
     <joint name="${arm_id}_joint6" type="revolute">

Commit message: description   : add world link

File: robots/polar_arm.xacro (robot description, xacro)
@@ -5,7 +5,7 @@
   <xacro:macro name="polar_arm" params="arm_id:='polar' description_pkg:='polar_description' connected_to:='' xyz:='0 0 0' rpy:='0 0 0'">
     <xacro:unless value="${not connected_to}">
-      <joint name="${arm_id}_joint_${connected_to}" type="fixed">
-        <parent link="${connected_to}"/>
-        <child link="${arm_id}_link0"/>
+      <joint name="virtual_joint" type="fixed">
+        <parent link="${connected_to}"/> <!-- world -->
+        <child link="${arm_id}_link0"/> <!-- base link -->
         <origin rpy="${rpy}" xyz="${xyz}"/>
       </joint>
@@ -16,10 +16,4 @@
     <xacro:property name="safety_k_velocity" value="40.0"/>
     <xacro:property name="safety_pos_margin" value="0.0"/>
-    <link name="world" />
-    <joint name="robot_to_world" type="fixed">
-      <parent link="world" />
-      <child link="${arm_id}_link0" />
-      <origin xyz="0.0 0.0 0.0" rpy="0.0 0.0 0.0" />
-    </joint>
     <link name="${arm_id}_link0">
       <visual>

File: robots/polar_arm_hand.urdf.xacro (robot description, xacro)
@@ -6,5 +6,6 @@
   <xacro:include filename="$(find polar_description)/robots/polar.gazebo.xacro"/>
   <xacro:include filename="$(find polar_description)/robots/polar.transmission.xacro"/>
-  <xacro:polar_arm/>
+  <link name="world" />
+  <xacro:polar_arm xyz="0 0 0" rpy="0 0 0" connected_to="world"/>
    <!-- Gripper description will be implemented -->
   <!-- <xacro:hand ns="polar" connected_to="polar_link6"/> -->
